Commit message: Trying to solve rviz error

File: Assignment2_exprob_TM/urdf/robot.xacro (robot description, xacro)
@@ -182,3 +182,27 @@
         <limit effort="10000" velocity="100" />
     </joint>
+    <link name="lidar_link">
+        <collision>
+            <origin xyz="0 0 0" rpy="0 0 0"/>
+            <geometry>
+                <cylinder length="0.05" radius="0.025"/>
+            </geometry>
+        </collision>
+        <visual>
+            <origin xyz="0 0 0.0" rpy="0 0 0"/>
+            <geometry>
+                <cylinder length="0.05" radius="0.025"/>
+            </geometry>
+            <material name="red">
+                <color rgba="1 0 0 1"/>
+            </material>
+        </visual>
+        <xacro:default_inertial mass="0.01"/>
+    </link>
+    <joint name="lidar_joint" type="fixed">
+        <parent link="link_chassis"/>
+        <child link="lidar_link"/>
+        <axis xyz="0 0 1" />
+        <origin xyz="0.20 0.0 0.05" rpy="0 0 0"/>
+    </joint>
 </robot>

Commit message: changed old remains

File: Assignment2_exprob_TM/urdf/robot.xacro (robot description, xacro)
@@ -1,5 +1,5 @@
 <?xml version="1.0"?>
 <robot xmlns:xacro="http://www.ros.org/wiki/xacro" name="robot">
-    <xacro:include filename="$(find exprob_dt)/urdf/robot.gazebo"/>
+    <xacro:include filename="$(find assignment2_exprob_tm)/urdf/robot.gazebo"/>
     <xacro:property name="length_wheel" value="0.04" />
     <xacro:property name="radius_wheel" value="0.1" />
@@ -87,20 +87,8 @@
         </visual>
     </link>
-    <link name="link_left_wheel">
-        <xacro:default_inertial mass="0.2"/>
-        <collision name="link_left_wheel_collision">
-            <origin rpy="0 1.5707 1.5707" xyz="0 0 0"/>
-            <xacro:wheel_geometry />
-        </collision>
-        <visual name="link_left_wheel_visual">
-            <origin rpy="0 1.5707 1.5707" xyz="0 0 0"/>
-            <xacro:wheel_geometry />
-            <material name="red"/>
-        </visual>
-    </link>
     <joint name="joint_right_wheel" type="continuous">
         <origin rpy="0 0 0" xyz="-0.05 0.15 0"/>
+        <parent link="link_chassis"/>
         <child link="link_right_wheel"/>
-        <parent link="link_chassis"/>
         <axis rpy="0 0 0" xyz="0 1 0"/>
         <limit effort="10000" velocity="1000"/>
@@ -108,11 +96,23 @@
     </joint>
     <joint name="joint_left_wheel" type="continuous">
+        <parent link="link_chassis"/>
+        <child link="link_left_wheel"/>
         <origin rpy="0 0 0" xyz="-0.05 -0.15 0"/>
-        <child link="link_left_wheel"/>
-        <parent link="link_chassis"/>
         <axis rpy="0 0 0" xyz="0 1 0"/>
         <limit effort="10000" velocity="1000"/>
         <joint_properties damping="1.0" friction="1.0"/>
     </joint>
+    <link name="link_left_wheel">
+        <xacro:default_inertial mass="0.2"/>
+        <collision>
+            <origin rpy="0 1.5707 1.5707" xyz="0 0 0"/>
+            <xacro:wheel_geometry/>
+        </collision>
+        <visual>
+            <origin rpy="0 1.5707 1.5707" xyz="0 0 0"/>
+            <xacro:wheel_geometry/>
+            <material name="red"/>
+        </visual>
+    </link>
     <link name="camera_optical_link">
         <inertial>
@@ -169,8 +169,8 @@
         <xacro:default_inertial mass="0.02"/>
         <!--<inertial>-->
-        <!--    <mass value="1e-5" />-->
-        <!--    <origin xyz="0 0 0" rpy="0 0 0"/>-->
-        <!--    <inertia ixx="1e-6" ixy="0" ixz="0" iyy="1e-6" iyz="0" izz="1e-6" />-->
-        <!--</inertial> -->
+            <!--    <mass value="1e-5" />-->
+            <!--    <origin xyz="0 0 0" rpy="0 0 0"/>-->
+            <!--    <inertia ixx="1e-6" ixy="0" ixz="0" iyy="1e-6" iyz="0" izz="1e-6" />-->
+            <!--</inertial> -->
     </link>
     <joint name="camera_joint" type="continuous">

Commit message: Recrated corect directory structure and odom

File: Assignment2_exprob_TM/urdf/robot.xacro (robot description, xacro)
@@ -42,8 +42,8 @@
     <link name="link_chassis">
         <!-- pose and inertial -->
-        <pose>0 0 0.1 0 0 0</pose>
+        <pose>0 0 0.0 0 0 0</pose>
         <inertial>
             <mass value="5"/>
-            <origin rpy="0 0 0" xyz="0 0 0.1"/>
+            <origin rpy="0 0 0" xyz="0 0 0.0"/>
             <inertia ixx="0.0395416666667" ixy="0" ixz="0" iyy="0.106208333333" iyz="0" izz="0.106208333333"/>
         </inertial>
@@ -178,5 +178,5 @@
         <child link="camera_connection_link"/>
         <axis xyz="0 0 1" />
-        <origin xyz="0.1 0.0 0.13" rpy="0 0 0"/>
+        <origin xyz="0.0 0.0 0.13" rpy="0 0 0"/>
         <dynamics damping="0.1"/>
         <limit effort="10000" velocity="100" />
@@ -206,3 +206,11 @@
         <origin xyz="0.20 0.0 0.05" rpy="0 0 0"/>
     </joint>
+    <link name="wheel_center_link">
+    </link>
+    <joint name="wheel_center_joint" type="fixed">
+        <origin rpy="0 0 0" xyz="-0.05 0 0"/>
+        <parent link="link_chassis"/>
+        <child link="wheel_center_link"/>
+        <axis rpy="0 0 0" xyz="0 1 0"/>
+    </joint>
 </robot>
