Commit message: First finished version

File: Assignment2_exprob_TM/urdf/test.urdf (robot description, URDF)
Before this commit: robot diff_robot, 8 links, 7 joints
Links:
- link left_wheel: mass 0.3 -> 0.8
- link lidar_link: mass 0.114 -> 0.004
- link right_wheel: mass 0.3 -> 0.8
Joints:
- joint base_camera_joint: origin xyz=0.0 0.0 0.18 rpy=0.0 0.0 0.0 -> xyz=0.2 0.0 0.17 rpy=0.0 0.0 0.0
- joint base_lidar_joint: origin xyz=0.0 0.0 0.08 rpy=0.0 0.0 0.0 -> xyz=0.2 0.0 0.08 rpy=0.0 0.0 0.0
